Commit message: [urdf] update wrench_sensor origin position in beetle_art_omni.urdf.xacro based on datasheet.

File: robots/beetle_omni/urdf/beetle_art_omni.urdf.xacro (robot description, xacro)
@@ -250,5 +250,5 @@
     <link name="wrench_sensor">
       <inertial>
-        <origin xyz="-0.00941317 0.00000000 -0.01652886" rpy="0 0 0"/>
+        <origin xyz="0.00000000 0.00000000 -0.01500000" rpy="0 0 0"/>
         <mass value="0.285"/>
         <inertia
