Commit message: [planning] valve manipulation migrating, [robot] change prismatic to ideal

File: robots/amoeba/urdf/amoeba.urdf.xacro (robot description, xacro)
@@ -92,10 +92,11 @@
       ## prismatic joint for chain_link arm
       <joint name="extendable_joint${id}" type="prismatic">
-        <limit effort="100.0" lower="-0.1" upper="0.1" velocity="0.01"/>
+        <!-- ideal prismatic -->
+        <limit effort="1000.0" lower="-0.1" upper="0.1" velocity="0.2"/>
         <parent link="rotor_arm${id}"/>
         <child link="chain_link${id}"/>
         <origin rpy="0 0 0" xyz="0 0 0"/>
         <axis xyz="1 0 0"/>
-        <dynamics damping="1.0" friction="0.1"/>
+        <dynamics damping="0.0" friction="0.0"/>
       </joint>
       ## transmission for extendable joint

Commit message: [robot]update amb2 [control] update gimbal name readable

File: robots/amoeba/urdf/amoeba.urdf.xacro (robot description, xacro)
@@ -7,9 +7,15 @@
     <link name="main_body">
       <inertial>
-        <origin xyz="-0.00034742 0.00036736 0.03608269" rpy="0 0 0"/>
-        <mass value="1.52925596"/>
-        <inertia
-            ixx="0.00714742" iyy=" 0.00722236" izz="0.00472163"
-            ixy="0.00000654" ixz=" 0.00015170" iyz="0.00005556"/>
+        <origin xyz="0.00058522 -0.00034768 0.02578334" rpy="0 0 0"/>
+        <mass value="1.39175439"/>
+        <inertia
+            ixx =" 0.00405786" iyy =" 0.00427970" izz =" 0.00420946"
+            ixy =" -0.00000961" ixz =" 0.00016759" iyz =" -0.00002723"/>
+        # battery
+        <!-- <origin xyz="0.00035664 -0.00021188 -0.00225415" rpy="0 0 0"/>
+        <mass value="2.28375439"/>
+        <inertia
+          ixx =" 0.00860275" iyy =" 0.00842374" izz =" 0.00708753"
+          ixy =" -0.00000972" ixz =" 0.00019043" iyz =" -0.00004080"/> -->
       </inertial>
       <visual>
@@ -69,9 +75,9 @@
       <link name="chain_link${id}">
         <inertial>
-          <origin xyz="-0.0917549 -0.000000 -0.0010835" rpy="0 0 0"/>
-          <mass value="0.1110974"/>
+          <origin xyz="-0.0679083 0.0000000 -0.0014430" rpy="0 0 0"/>
+          <mass value="0.1143400"/>
           <inertia
-              ixx="0.0000194" ixy="0.0" ixz="-0.0000107"
-              iyy="0.0004353" iyz="0.0" izz="0.0004368"/>
+              ixx ="  0.0000329" iyy ="0.0003105" izz =" 0.0003140"
+              ixy =" 0.0000000" ixz ="-0.0000088" iyz =" 0.0000000"/>
         </inertial>
         <!-- the motor_case's limit pin is 87mm from the servo -->
@@ -154,8 +160,8 @@
     </xacro:macro>
     ## dummy rotor arms
-    <xacro:dummy_rotor_arm id = "${child1}" x = " 0.198956" y=" 0.198956" z = "0.0154" yaw = "${pi*1.0/4.0}"/>
-    <xacro:dummy_rotor_arm id = "${child2}" x = "-0.198956" y=" 0.198956" z = "0.0154" yaw = "${pi*3.0/4.0}"/>
-    <xacro:dummy_rotor_arm id = "${child3}" x = "-0.198956" y="-0.198956" z = "0.0154" yaw = "${pi*5.0/4.0}"/>
-    <xacro:dummy_rotor_arm id = "${child4}" x = " 0.198956" y="-0.198956" z = "0.0154" yaw = "${-pi*1.0/4.0}"/>
+    <xacro:dummy_rotor_arm id = "${child1}" x = " 0.150755" y=" 0.150755" z = "0.0175" yaw = "${pi*1.0/4.0}"/>
+    <xacro:dummy_rotor_arm id = "${child2}" x = "-0.150755" y=" 0.150755" z = "0.0175" yaw = "${pi*3.0/4.0}"/>
+    <xacro:dummy_rotor_arm id = "${child3}" x = "-0.150755" y="-0.150755" z = "0.0175" yaw = "${pi*5.0/4.0}"/>
+    <xacro:dummy_rotor_arm id = "${child4}" x = " 0.150755" y="-0.150755" z = "0.0175" yaw = "${-pi*1.0/4.0}"/>
     <xacro:friction self="main_body"/>
   </xacro:macro>
@@ -165,9 +171,9 @@
     <link name="gimbal_link${self}">
       <inertial>
-        <origin xyz="0.02786199 -0.00000778 -0.01385805" rpy="0 0 0"/>
-        <mass value="0.1702000"/>
-        <inertia
-            ixx="0.00017696" iyy="0.00018593" izz="0.00027041"
-            ixy="0.00000002" ixz="-0.00002708" iyz="0.0"/>
+        <origin xyz="0.07576614 0.00018422 0.00143736" rpy="0 0 0"/>
+        <mass value="0.17880658"/>
+        <inertia
+            ixx =" 0.00019959" iyy =" 0.00028405" izz =" 0.00038626"
+            ixy =" -0.00000220" ixz = "0.00000178" iyz ="-0.00000004"/>
       </inertial>
       <collision>
@@ -232,5 +238,5 @@
       <parent link="gimbal_link${self}"/>
       <child link="rotor_parent${self}"/>
-      <origin rpy="0 0 0" xyz="0.02185 0.0 0.0"/>
+      <origin rpy="0 0 0" xyz="0.083 0.0 0.0"/>
     </joint>
     #### rotor joint (virtual) ####

Commit message: [robot] update fc position

File: robots/amoeba/urdf/amoeba.urdf.xacro (robot description, xacro)
@@ -51,5 +51,5 @@
       <child link="fc"/>
       <parent link="main_body"/>
-      <origin rpy="0 0 0" xyz="-0.0175 -0.0015 0.06347"/>  # should be aligned with the position of IMU
+      <origin rpy="0 0 0" xyz="-0.0175 -0.0015 0.06047"/>  # should be aligned with the position of IMU
       <!-- changed from omni to amoeba -->
     </joint>

Commit message: [amoeba] upadate collision and spawn point

File: robots/amoeba/urdf/amoeba.urdf.xacro (robot description, xacro)
@@ -26,7 +26,7 @@
       </visual>
       <collision>
-        <origin xyz="0 0 0.0385" rpy="0 0 ${pi/4}"/>
-        <geometry>
-          <box size="0.12 0.12 0.275"/>
+        <origin xyz="0 0 0.0335" rpy="0 0 ${pi/4}"/>
+        <geometry>
+          <box size="0.12 0.12 0.225"/>
         </geometry>
       </collision>

Commit message: [amoeba] update thrust and weight

File: robots/amoeba/urdf/amoeba.urdf.xacro (robot description, xacro)
@@ -8,14 +8,8 @@
       <inertial>
         <origin xyz="0.00058522 -0.00034768 0.02578334" rpy="0 0 0"/>
-        <mass value="1.39175439"/>
+        <mass value="1.49175439"/>
         <inertia
             ixx =" 0.00405786" iyy =" 0.00427970" izz =" 0.00420946"
             ixy =" -0.00000961" ixz =" 0.00016759" iyz =" -0.00002723"/>
-        # battery
-        <!-- <origin xyz="0.00035664 -0.00021188 -0.00225415" rpy="0 0 0"/>
-        <mass value="2.28375439"/>
-        <inertia
-          ixx =" 0.00860275" iyy =" 0.00842374" izz =" 0.00708753"
-          ixy =" -0.00000972" ixz =" 0.00019043" iyz =" -0.00004080"/> -->
       </inertial>
       <visual>

File: robots/amoeba/urdf/common.xacro (robot description, xacro)
@@ -5,5 +5,5 @@
   <thrust_link name="thrust" />
   <m_f_rate value="-0.0165" /> <!-- drag torque rate -->
-  <xacro:property name="max_force" value="30.0" /> <!-- [N] -->
+  <xacro:property name="max_force" value="19.0" /> <!-- [N] -->
   <xacro:property name="min_force" value="1.0" /> <!-- [N] -->
   <!-- friction -->

Commit message: [amoeba] upadate inertia with battery

File: robots/amoeba/urdf/amoeba.urdf.xacro (robot description, xacro)
@@ -7,9 +7,19 @@
     <link name="main_body">
       <inertial>
-        <origin xyz="0.00058522 -0.00034768 0.02578334" rpy="0 0 0"/>
-        <mass value="1.49175439"/>
-        <inertia
-            ixx =" 0.00405786" iyy =" 0.00427970" izz =" 0.00420946"
-            ixy =" -0.00000961" ixz =" 0.00016759" iyz =" -0.00002723"/>
+        <xacro:unless value="${battery == 1}">
+          <origin xyz="0.01558522 -0.00034768 0.02578334" rpy="0 0 0"/>
+          <mass value="1.49175439"/>
+          <inertia
+              ixx =" 0.00405786" iyy =" 0.00427970" izz =" 0.00420946"
+              ixy =" -0.00000961" ixz =" 0.00016759" iyz =" -0.00002723"/>
+        </xacro:unless>
+        <xacro:if value="${battery == 1}">
+          <!-- with battery -->
+          <origin xyz="0.00035664 -0.00021188 -0.00225415" rpy="0 0 0"/>
+          <mass value="2.28375439"/>
+          <inertia
+              ixx =" 0.00860275" iyy =" 0.00842374" izz =" 0.00708753"
+              ixy =" -0.00000972" ixz =" 0.00019043" iyz =" -0.00004080"/>
+        </xacro:if>
       </inertial>
       <visual>
@@ -20,7 +30,7 @@
       </visual>
       <collision>
-        <origin xyz="0 0 0.0335" rpy="0 0 ${pi/4}"/>
-        <geometry>
-          <box size="0.12 0.12 0.225"/>
+        <origin xyz="0 0 0.0135" rpy="0 0 ${pi/4}"/>
+        <geometry>
+          <box size="0.12 0.12 0.185"/>
         </geometry>
       </collision>
@@ -255,4 +265,6 @@
 <!-- Define beetle -->
   <xacro:arg name="robot_name" default="beetle-art-omni" />
+  <xacro:arg name="battery" default="0" />
+  <xacro:property name="battery" value="$(arg battery)" />
   <xacro:beetle_center_link child1="1" child2="2" child3="3" child4="4"/>
   <xacro:beetle_thrust_link self="1" rotor_direction="1"/>
@@ -271,5 +283,5 @@
     <parent link="main_body"/>
     <child link="end"/>
-    <origin xyz="0 0 0.1725" rpy="0 0 0"/>
+    <origin xyz="0 0 0.106" rpy="0 0 0"/>
   </joint>
   <!-- Conditionally create the fork or ball link based on the parameter value -->
