Commit message: [robot]update battery inertia

File: robots/amoeba/urdf/amoeba.urdf.xacro (robot description, xacro)
@@ -16,6 +16,6 @@
         <xacro:if value="${battery == 1}">
           <!-- with battery -->
-          <origin xyz="0.00035664 -0.00021188 -0.00225415" rpy="0 0 0"/>
-          <mass value="2.28375439"/>
+          <origin xyz="0.0025 0.0 -0.00225415" rpy="0 0 0"/>
+          <mass value="2.35"/>
           <inertia
               ixx =" 0.00860275" iyy =" 0.00842374" izz =" 0.00708753"

Commit message: [robot] add D435i model and view

File: robots/amoeba/urdf/amoeba.urdf.xacro (robot description, xacro)
@@ -1,4 +1,5 @@
 <?xml version="1.0"?>
 <robot xmlns:xacro="http://www.ros.org/wiki/xacro" name="beetle_link" >
+  <xacro:include filename="$(find amoeba)/urdf/sensors/d435i.xacro" />
   <xacro:macro name="beetle_center_link" params="child1 child2 child3 child4">
     ## dummy
@@ -266,5 +267,7 @@
   <xacro:arg name="robot_name" default="beetle-art-omni" />
   <xacro:arg name="battery" default="0" />
+  <xacro:arg name="enable_d435i" default="false" />
   <xacro:property name="battery" value="$(arg battery)" />
+  <xacro:property name="enable_d435i" value="$(arg enable_d435i)" />
   <xacro:beetle_center_link child1="1" child2="2" child3="3" child4="4"/>
   <xacro:beetle_thrust_link self="1" rotor_direction="1"/>
@@ -285,4 +288,11 @@
     <origin xyz="0 0 0.106" rpy="0 0 0"/>
   </joint>
+  <xacro:if value="${enable_d435i}">
+    <xacro:d435i_depth_camera
+        parent_link="main_body"
+        robot_ns="$(arg robot_name)"
+        xyz="-0.02 -0.02 0.106"
+        rpy="0 ${-pi * 9.0 / 180.0} ${pi * 5.0 / 4.0}"/>
+  </xacro:if>
   <!-- Conditionally create the fork or ball link based on the parameter value -->
   <xacro:if value="${end_effector == 'fork'}">

Commit message: [robot]add amoeba duct_perch

File: robots/amoeba/urdf/amoeba.urdf.xacro (robot description, xacro)
@@ -175,9 +175,18 @@
     <link name="gimbal_link${self}">
       <inertial>
-        <origin xyz="0.07576614 0.00018422 0.00143736" rpy="0 0 0"/>
-        <mass value="0.17880658"/>
-        <inertia
-            ixx =" 0.00019959" iyy =" 0.00028405" izz =" 0.00038626"
-            ixy =" -0.00000220" ixz = "0.00000178" iyz ="-0.00000004"/>
+        <xacro:if value="${self == 1 or self == 3}">
+          <origin xyz="0.07576614 0.00018422 0.00143736" rpy="0 0 0"/>
+          <mass value="0.17880658"/>
+          <inertia
+              ixx =" 0.00019959" iyy =" 0.00028405" izz =" 0.00038626"
+              ixy =" -0.00000220" ixz = "0.00000178" iyz ="-0.00000004"/>
+        </xacro:if>
+        <xacro:if value="${self == 2 or self == 4}">
+          <origin xyz="0.08674561 -0.00074 0.04888743" rpy="0 0 0"/>
+          <mass value="0.22136000"/>
+          <inertia
+              ixx ="0.00094603" iyy ="0.00281080" izz ="0.00276983"
+              ixy ="-0.00001486" ixz ="0.00026438" iyz ="-0.00000586"/>
+        </xacro:if>
       </inertial>
       <collision>

Commit message: [robot] update grasper

File: robots/amoeba/urdf/amoeba.urdf.xacro (robot description, xacro)
@@ -79,9 +79,18 @@
       <link name="chain_link${id}">
         <inertial>
-          <origin xyz="-0.0679083 0.0000000 -0.0014430" rpy="0 0 0"/>
-          <mass value="0.1143400"/>
-          <inertia
-              ixx ="  0.0000329" iyy ="0.0003105" izz =" 0.0003140"
-              ixy =" 0.0000000" ixz ="-0.0000088" iyz =" 0.0000000"/>
+          <xacro:if value="${id == 1 or id == 3}">
+            <origin xyz=" -0.0673206 0.0000000 -0.0014430" rpy="0 0 0"/>
+            <mass value="0.1139600"/>
+            <inertia
+                ixx =" 0.0000325" iyy =" 0.0003041" izz =" 0.0003080"
+                ixy =" 0.0000000" ixz =" -0.0000087" iyz =" 0.0000000"/>
+          </xacro:if>
+          <xacro:if value="${id == 2 or id == 4}">
+            <origin xyz="-0.0565922 0.0000183 -0.0266963" rpy="0 0 0"/>
+            <mass value="0.1569763"/>
+            <inertia
+                ixx =" 0.0003726" iyy ="0.0006876" izz =" 0.0003903"
+                ixy =" 0.0000001" ixz ="-0.0001248" iyz ="-0.0000002"/>
+          </xacro:if>
         </inertial>
         <!-- the motor_case's limit pin is 87mm from the servo -->
